File: Hardware/Micro-OLED_I2C.brd (EAGLE design)
At the start: 20.3 x 29.2 mm, 26 parts

Commit message: More mold modifications Elongated the PCB for mold
Other:
- board text removed: "Jim Lindblom"
