File: Hardware/Qwiic_OLED_Breakout.sch (EAGLE design)
At the start: 25 parts

Commit message: Mold V2
Parts:
- removed JP1: JUMPER-SMT_3_1-NC_PASTE_SILK, SparkFun-Jumpers:JUMPER-SMT_3_1-NC_PASTE_SILK
- added JP3: JUMPER-SMT_2_NO_SILK, SparkFun-Jumpers:JUMPER-SMT_2_NO_SILK
- added U$3: SPARKX-LOGO2, SparkX:SPARKX-LOGO2
Connections:
- removed net VDD_PU1: JP1.3, OLED1.BS1, R3.1
- net D/C: now also JP3.2, R3.1; no longer JP1.2
- net GND: now also JP3.1; no longer JP1.1
- net VDD: now also OLED1.BS1
Other:
- note added: "Joel Bartlett"
- note added: "X10"
- note removed: "v04"
- moved on the sheet: R3
Changed lines of the file:
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@@
 <part name="GND7" library="SparkFun-Aesthetics" deviceset="GND" device=""/>
 <part name="GND22" library="SparkFun-Aesthetics" deviceset="GND" device=""/>
-<part name="JP1" library="SparkFun-Jumpers" deviceset="JUMPER-SMT_3_1-NC_PASTE" device="_SILK" value="JUMPER-SMT_3_1-NC_PASTE_SILK"/>
 <part name="R13" library="SparkFun-Resistors" deviceset="4.7KOHM" device="-0603-1/10W-1%" value="4.7k"/>
 <part name="R14" library="SparkFun-Resistors" deviceset="4.7KOHM" device="-0603-1/10W-1%" value="4.7k"/>
@@
 <part name="H2" library="SparkFun-Hardware" deviceset="STAND-OFF" device=""/>
 <part name="SUPPLY2" library="SparkFun-Aesthetics" deviceset="VDD" device=""/>
+<part name="JP3" library="SparkFun-Jumpers" deviceset="JUMPER-SMT_2_NO" device="_SILK" value=""/>
+<part name="SUPPLY9" library="SparkFun-Aesthetics" deviceset="VDD" device=""/>
+<part name="U$3" library="SparkX" deviceset="SPARKX-LOGO" device="2"/>
 </parts>
 <sheets>
 <sheet>
 <plain>
-<text x="239.014" y="6.604" size="3.81" layer="94">v04</text>
+<text x="236.982" y="6.35" size="3.81" layer="94">X10</text>
 <text x="178.816" y="150.876" size="1.778" layer="97">1.65 &lt;= VDD &lt;= 3.3</text>
 <text x="195.58" y="129.54" size="1.778" layer="97">VDD current &lt; 300 uA</text>
@@
 then pulls HIGH once capacitor is charged
 after 10ms</text>
-<text x="149.86" y="96.52" size="1.778" layer="97">BS1 is pulled HIGH and
+<text x="48.26" y="83.82" size="1.778" layer="97">BS1 is pulled HIGH and
 BS@ is Pulled LOW for
 permanent I2C mode.</text>
@@
 to 4.7k pull-up
 resistors.</text>
+<text x="171.196" y="11.176" size="2.54" layer="94">Joel Bartlett</text>
 </plain>
 <instances>
@@
 <instance part="GND13" gate="1" x="25.4" y="78.74"/>
 <instance part="U$1" gate="G$1" x="134.62" y="5.08"/>
-<instance part="R3" gate="G$1" x="78.74" y="86.36" rot="MR90"/>
-<instance part="SUPPLY8" gate="VDD" x="78.74" y="93.98" rot="MR0"/>
+<instance part="R3" gate="G$1" x="157.48" y="88.9" rot="MR90"/>
+<instance part="SUPPLY8" gate="VDD" x="157.48" y="96.52" rot="MR0"/>
 <instance part="C7" gate="G$1" x="20.32" y="144.78"/>
 <instance part="R2" gate="G$1" x="12.7" y="154.94"/>
@@
 <instance part="GND7" gate="1" x="20.32" y="137.16"/>
 <instance part="GND22" gate="1" x="157.48" y="60.96" rot="MR0"/>
-<instance part="JP1" gate="G$1" x="157.48" y="71.12" rot="R180"/>
 <instance part="R13" gate="G$1" x="53.34" y="147.32" rot="R90"/>
 <instance part="R14" gate="G$1" x="68.58" y="147.32" rot="R90"/>
@@
 <instance part="H2" gate="G$1" x="238.76" y="33.02"/>
 <instance part="SUPPLY2" gate="VDD" x="60.96" y="165.1"/>
+<instance part="JP3" gate="G$1" x="157.48" y="71.12" rot="R90"/>
+<instance part="SUPPLY9" gate="VDD" x="86.36" y="81.28" rot="MR0"/>
+<instance part="U$3" gate="G$1" x="134.62" y="5.08"/>
 </instances>
 <busses>
@@
 <pinref part="GND22" gate="1" pin="GND"/>
 <wire x1="157.48" y1="63.5" x2="157.48" y2="66.04" width="0.1524" layer="91"/>
-<pinref part="JP1" gate="G$1" pin="1"/>
+<pinref part="JP3" gate="G$1" pin="1"/>
 </segment>
 </net>
@@
 <pinref part="R3" gate="G$1" pin="2"/>
 <pinref part="SUPPLY8" gate="VDD" pin="VDD"/>
-<wire x1="78.74" y1="93.98" x2="78.74" y2="91.44" width="0.1524" layer="91"/>
+<wire x1="157.48" y1="96.52" x2="157.48" y2="93.98" width="0.1524" layer="91"/>
 </segment>
 <segment>
@@
 <pinref part="SUPPLY2" gate="VDD" pin="VDD"/>
 <wire x1="60.96" y1="165.1" x2="60.96" y2="162.56" width="0.1524" layer="91"/>
+</segment>
+<segment>
+<pinref part="OLED1" gate="G1" pin="BS1"/>
+<wire x1="96.52" y1="68.58" x2="86.36" y2="68.58" width="0.1524" layer="91"/>
+<pinref part="SUPPLY9" gate="VDD" pin="VDD"/>
+<wire x1="86.36" y1="81.28" x2="86.36" y2="68.58" width="0.1524" layer="91"/>
 </segment>
 </net>
@@
 </segment>
 <segment>
-<wire x1="162.56" y1="71.12" x2="165.1" y2="71.12" width="0.1524" layer="91"/>
-<label x="165.1" y="71.12" size="1.27" layer="95" rot="MR180" xref="yes"/>
-<pinref part="JP1" gate="G$1" pin="2"/>
-</segment>
-</net>
-<net name="VDD_PU1" class="0">
-<segment>
-<wire x1="157.48" y1="76.2" x2="157.48" y2="83.82" width="0.1524" layer="91"/>
-<wire x1="157.48" y1="83.82" x2="162.56" y2="83.82" width="0.1524" layer="91"/>
-<label x="162.56" y="83.82" size="1.27" layer="95" xref="yes"/>
-<pinref part="JP1" gate="G$1" pin="3"/>
-</segment>
-<segment>
-<pinref part="OLED1" gate="G1" pin="BS1"/>
-<wire x1="96.52" y1="68.58" x2="78.74" y2="68.58" width="0.1524" layer="91"/>
-<label x="76.2" y="68.58" size="1.27" layer="95" rot="R180" xref="yes"/>
+<label x="162.56" y="78.74" size="1.27" layer="95" rot="MR180" xref="yes"/>
+<pinref part="JP3" gate="G$1" pin="2"/>
+<wire x1="162.56" y1="78.74" x2="157.48" y2="78.74" width="0.1524" layer="91"/>
+<wire x1="157.48" y1="78.74" x2="157.48" y2="76.2" width="0.1524" layer="91"/>
 <pinref part="R3" gate="G$1" pin="1"/>
-<wire x1="78.74" y1="68.58" x2="76.2" y2="68.58" width="0.1524" layer="91"/>
-<wire x1="78.74" y1="81.28" x2="78.74" y2="68.58" width="0.1524" layer="91"/>
-<junction x="78.74" y="68.58"/>
-</segment>
-</net>
+<wire x1="157.48" y1="83.82" x2="157.48" y2="78.74" width="0.1524" layer="91"/>
+<junction x="157.48" y="78.74"/>
+</segment>
+</net>
