File: Hardware/Qwiic_OLED_Breakout_NO_T.brd (EAGLE design)
At the start: 27.3 x 29.2 mm, 27 parts

Commit message: Adding Gerbers
Parts:
- removed H1, H2: STAND-OFF, SparkFun-Hardware:STAND-OFF
- removed U$1, U$2: SPARKX-LOGO4, SparkX:SPARKX-MEDIUM
- moved FRAME1 36.7 mm to (17.8, -19.1), flipped to the bottom
Other:
- board size 27.3 x 29.2 mm -> 20.3 x 29.1 mm
- board text removed: "Joel Bartlett"
